Commit message: Modify bot to use a single caster wheel instead

File: src/description/base-bot-2.urdf (robot description, URDF)
Before this commit: robot differential-bot, 2 links, 1 joints
Links:
- added link caster_whl; visual sphere radius=${-(wheel_radius+wheel_zoff-(base_height/2))}
- link base_link: geometry visual box size=${base_length} ${base_width} ${base_height}
Joints:
- added joint caster_joint: type fixed, parent base_link, child caster_whl, origin xyz=${wheel_xoff} 0.0 ${-(base_height/2)} rpy=0 0 0

Commit message: Add physical properties and tweak dimensions

File: src/description/base-bot-2.urdf (robot description, URDF)
Before this commit: robot differential-bot, 3 links, 2 joints
Links:
- link base_link: geometry collision box size=${base_length} ${base_width} ${base_height}; visual box size=${base_length} ${base_width} ${base_height}
- link caster_whl: geometry collision sphere radius=${-(wheel_radius+wheel_zoff-(base_height/2))}; visual sphere radius=${-(wheel_radius+wheel_zoff-(base_height/2))}
Joints:
- joint caster_joint: origin xyz=${wheel_xoff} 0.0 ${-(base_height/2)} rpy=0 0 0 -> xyz=${caster_xoff} 0.0 ${-(base_height/2)} rpy=0 0 0
