Commit message: Rename project, caster wheels and robot

File: src/description/sam-bot_description.urdf (robot description, URDF)
Before this commit: robot differential-bot, 3 links, 2 joints
Links:
- removed link caster_whl
- added link front_caster; collision sphere radius=${-(wheel_radius+wheel_zoff-(base_height/2))}; visual sphere radius=${-(wheel_radius+wheel_zoff-(base_height/2))}
Joints:
- joint caster_joint: child caster_whl -> front_caster
